Commit message: add gripper control support
position_controllers/GripperActionController is implemented for now yet parallel_gripper_controller/GripperActionController is recommended for Jazzy+.

Signed-off-by: Baoan Du <baoan.du.xj@renesas.com>

File: urdf/agilex_piper_arm.urdf.xacro (robot description, xacro)
@@ -18,4 +18,5 @@
     name="AgilexPiperSystem"
     can_interface="$(arg can_interface)"
-    use_mock_hardware="$(arg use_mock_hardware)"/>
+    use_mock_hardware="$(arg use_mock_hardware)"
+    include_gripper="false"/>
 </robot>

File: urdf/agilex_piper_ros2_control.xacro (robot description, xacro)
@@ -39,8 +39,25 @@
     </joint>
   </xacro:macro>
+  <!-- Gripper interface definitions -->
+  <xacro:macro name="piper_gripper_interfaces">
+    <!-- Both joints need to be controlled for proper visualization -->
+    <joint name="joint7">
+      <command_interface name="position"/>
+      <command_interface name="effort"/>
+      <state_interface name="position"/>
+      <state_interface name="velocity"/>
+    </joint>
+    <joint name="joint8">
+      <command_interface name="position"/>
+      <command_interface name="effort"/>
+      <state_interface name="position"/>
+      <state_interface name="velocity"/>
+    </joint>
+  </xacro:macro>
   <xacro:macro name="agilex_piper_ros2_control" params="
     name:=AgilexPiperSystem
     can_interface:=can0
-    use_mock_hardware:=false">
+    use_mock_hardware:=false
+    include_gripper:=true">
     <!-- Real hardware configuration -->
     <xacro:unless value="${use_mock_hardware}">
@@ -49,7 +66,12 @@
           <plugin>agilex_piper_ros2_control/AgilexPiperHardwareInterface</plugin>
           <param name="can_interface">${can_interface}</param>
+          <param name="include_gripper">${include_gripper}</param>
         </hardware>
         <!-- Joint interfaces -->
         <xacro:piper_joint_interfaces/>
+        <!-- Gripper interfaces (conditional) -->
+        <xacro:if value="${include_gripper}">
+          <xacro:piper_gripper_interfaces/>
+        </xacro:if>
       </ros2_control>
     </xacro:unless>
@@ -63,4 +85,8 @@
         <!-- Joint interfaces -->
         <xacro:piper_joint_interfaces/>
+        <!-- Gripper interfaces (conditional) -->
+        <xacro:if value="${include_gripper}">
+          <xacro:piper_gripper_interfaces/>
+        </xacro:if>
       </ros2_control>
     </xacro:if>

Commit message: Refactor ros2_control configuration to support dynamic prefix
Signed-off-by: Baoan Du <baoan.du.xj@renesas.com>

File: urdf/agilex_piper_arm.urdf.xacro (robot description, xacro)
@@ -4,4 +4,5 @@
   <xacro:arg name="can_interface" default="can0"/>
   <xacro:arg name="use_mock_hardware" default="false"/>
+  <xacro:arg name="prefix" default=""/>
   <!-- Include the arm description -->
   <xacro:include filename="$(find agilex_piper_arm_description)/urdf/agilex_piper_arm_macro.xacro"/>
@@ -11,12 +12,13 @@
   <link name="world"/>
   <!-- Mount the arm to world -->
-  <xacro:agilex_piper_arm prefix="" parent="world">
+  <xacro:agilex_piper_arm prefix="$(arg prefix)" parent="world">
     <origin xyz="0 0 0" rpy="0 0 0"/>
   </xacro:agilex_piper_arm>
   <!-- Add ros2_control -->
   <xacro:agilex_piper_ros2_control
-    name="AgilexPiperSystem"
+    name="agilex_piper_arm"
     can_interface="$(arg can_interface)"
     use_mock_hardware="$(arg use_mock_hardware)"
-    include_gripper="false"/>
+    include_gripper="false"
+    prefix="$(arg prefix)"/>
 </robot>

File: urdf/agilex_piper_arm_gripper.urdf.xacro (robot description, xacro)
@@ -4,4 +4,5 @@
   <xacro:arg name="can_interface" default="can0"/>
   <xacro:arg name="use_mock_hardware" default="false"/>
+  <xacro:arg name="prefix" default=""/>
   <!-- Include the arm description -->
   <xacro:include filename="$(find agilex_piper_arm_description)/urdf/agilex_piper_arm_macro.xacro"/>
@@ -13,16 +14,17 @@
   <link name="world"/>
   <!-- Mount the arm to world -->
-  <xacro:agilex_piper_arm prefix="" parent="world">
+  <xacro:agilex_piper_arm prefix="$(arg prefix)" parent="world">
     <origin xyz="0 0 0" rpy="0 0 0"/>
   </xacro:agilex_piper_arm>
   <!-- Mount the gripper to the arm's tool0 link -->
-  <xacro:agilex_piper_gripper prefix="" parent="tool0">
+  <xacro:agilex_piper_gripper prefix="$(arg prefix)" parent="$(arg prefix)tool0">
     <origin xyz="0 0 0" rpy="0 0 0"/>
   </xacro:agilex_piper_gripper>
   <!-- Add ros2_control -->
   <xacro:agilex_piper_ros2_control
-    name="AgilexPiperSystem"
+    name="agilex_piper_arm"
     can_interface="$(arg can_interface)"
     use_mock_hardware="$(arg use_mock_hardware)"
-    include_gripper="true"/>
+    include_gripper="true"
+    prefix="$(arg prefix)"/>
 </robot>

File: urdf/agilex_piper_macro.ros2_control.xacro (robot description, xacro)
@@ -6,89 +6,71 @@
     Supports both real hardware and mock hardware configurations
   -->
-  <!-- Shared joint interface definitions -->
-  <xacro:macro name="piper_joint_interfaces">
-    <joint name="joint1">
-      <command_interface name="position"/>
-      <state_interface name="position"/>
-      <state_interface name="velocity"/>
-    </joint>
-    <joint name="joint2">
-      <command_interface name="position"/>
-      <state_interface name="position"/>
-      <state_interface name="velocity"/>
-    </joint>
-    <joint name="joint3">
-      <command_interface name="position"/>
-      <state_interface name="position"/>
-      <state_interface name="velocity"/>
-    </joint>
-    <joint name="joint4">
-      <command_interface name="position"/>
-      <state_interface name="position"/>
-      <state_interface name="velocity"/>
-    </joint>
-    <joint name="joint5">
-      <command_interface name="position"/>
-      <state_interface name="position"/>
-      <state_interface name="velocity"/>
-    </joint>
-    <joint name="joint6">
-      <command_interface name="position"/>
-      <state_interface name="position"/>
-      <state_interface name="velocity"/>
-    </joint>
-  </xacro:macro>
-  <!-- Gripper interface definitions -->
-  <xacro:macro name="piper_gripper_interfaces">
-    <!-- Both joints need to be controlled for proper visualization -->
-    <joint name="joint7">
-      <command_interface name="position"/>
-      <command_interface name="effort"/>
-      <state_interface name="position"/>
-      <state_interface name="velocity"/>
-    </joint>
-    <joint name="joint8">
-      <command_interface name="position"/>
-      <command_interface name="effort"/>
-      <state_interface name="position"/>
-      <state_interface name="velocity"/>
-    </joint>
-  </xacro:macro>
   <xacro:macro name="agilex_piper_ros2_control" params="
-    name:=AgilexPiperSystem
+    name:=agilex_piper_arm
     can_interface:=can0
     use_mock_hardware:=false
-    include_gripper:=true">
-    <!-- Real hardware configuration -->
-    <xacro:unless value="${use_mock_hardware}">
-      <ros2_control name="${name}" type="system" rw_rate="100">
-        <hardware>
+    include_gripper:=true
+    prefix:=''
+    ">
+    <ros2_control name="${prefix}${name}" type="system" rw_rate="100">
+      <!-- Hardware interface plugin chosen conditionally -->
+      <hardware>
+        <xacro:if value="${use_mock_hardware}">
+          <plugin>mock_components/GenericSystem</plugin>
+          <param name="calculate_dynamics">true</param>
+        </xacro:if>
+        <xacro:unless value="${use_mock_hardware}">
           <plugin>agilex_piper_ros2_control/AgilexPiperHardwareInterface</plugin>
           <param name="can_interface">${can_interface}</param>
           <param name="include_gripper">${include_gripper}</param>
-        </hardware>
-        <!-- Joint interfaces -->
-        <xacro:piper_joint_interfaces/>
-        <!-- Gripper interfaces (conditional) -->
-        <xacro:if value="${include_gripper}">
-          <xacro:piper_gripper_interfaces/>
-        </xacro:if>
-      </ros2_control>
-    </xacro:unless>
-    <!-- Mock hardware configuration -->
-    <xacro:if value="${use_mock_hardware}">
-      <ros2_control name="${name}MockSystem" type="system">
-        <hardware>
-          <plugin>mock_components/GenericSystem</plugin>
-          <param name="calculate_dynamics">true</param>
-        </hardware>
-        <!-- Joint interfaces -->
-        <xacro:piper_joint_interfaces/>
-        <!-- Gripper interfaces (conditional) -->
-        <xacro:if value="${include_gripper}">
-          <xacro:piper_gripper_interfaces/>
-        </xacro:if>
-      </ros2_control>
-    </xacro:if>
+        </xacro:unless>
+      </hardware>
+      <!-- Joint definitions -->
+      <joint name="${prefix}joint1">
+        <command_interface name="position"/>
+        <state_interface name="position"/>
+        <state_interface name="velocity"/>
+      </joint>
+      <joint name="${prefix}joint2">
+        <command_interface name="position"/>
+        <state_interface name="position"/>
+        <state_interface name="velocity"/>
+      </joint>
+      <joint name="${prefix}joint3">
+        <command_interface name="position"/>
+        <state_interface name="position"/>
+        <state_interface name="velocity"/>
+      </joint>
+      <joint name="${prefix}joint4">
+        <command_interface name="position"/>
+        <state_interface name="position"/>
+        <state_interface name="velocity"/>
+      </joint>
+      <joint name="${prefix}joint5">
+        <command_interface name="position"/>
+        <state_interface name="position"/>
+        <state_interface name="velocity"/>
+      </joint>
+      <joint name="${prefix}joint6">
+        <command_interface name="position"/>
+        <state_interface name="position"/>
+        <state_interface name="velocity"/>
+      </joint>
+      <!-- Gripper definitions (conditional) -->
+      <xacro:if value="${include_gripper}">
+        <joint name="${prefix}joint7">
+          <command_interface name="position"/>
+          <command_interface name="effort"/>
+          <state_interface name="position"/>
+          <state_interface name="velocity"/>
+        </joint>
+        <joint name="${prefix}joint8">
+          <command_interface name="position"/>
+          <command_interface name="effort"/>
+          <state_interface name="position"/>
+          <state_interface name="velocity"/>
+        </joint>
+      </xacro:if>
+    </ros2_control>
   </xacro:macro>
 </robot>
